File: EAGLE/ADDON/230V2LED.brd (EAGLE design)
At the start: 15.2 x 35.6 mm, 10 parts

Commit message: move 230V2LED -> addon dir
Parts:
- R5: value (none) -> 22K
Routing:
- net N$9: track 25.4 -> 26.0 mm, vias 2 -> 4
Changed lines of the file:
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@@
 <?xml version="1.0" encoding="utf-8"?>
 <!DOCTYPE eagle SYSTEM "eagle.dtd">
-<eagle version="6.2">
+<eagle version="6.3">
 <drawing>
 <settings>
@@
 <layer number="25" name="tNames" color="7" fill="1" visible="no" active="yes"/>
 <layer number="26" name="bNames" color="7" fill="1" visible="no" active="yes"/>
-<layer number="27" name="tValues" color="7" fill="1" visible="no" active="yes"/>
+<layer number="27" name="tValues" color="7" fill="1" visible="yes" active="yes"/>
 <layer number="28" name="bValues" color="7" fill="1" visible="no" active="yes"/>
 <layer number="29" name="tStop" color="7" fill="3" visible="no" active="yes"/>
@@
 </class>
 </classes>
-<designrules>
+<designrules name="default">
 <description language="de">&lt;b&gt;EAGLE Design Rules&lt;/b&gt;
 &lt;p&gt;
@@
 <element name="R2" library="resistor" package="0207/2V" value="22K" x="3.81" y="12.7"/>
 <element name="JP2" library="pinhead" package="1X05" value="" x="7.62" y="30.48"/>
-<element name="R5" library="resistor" package="0207/2V" value="" x="6.35" y="33.02"/>
+<element name="R5" library="resistor" package="0207/2V" value="22K" x="6.35" y="33.02"/>
 <element name="R1" library="resistor" package="0207/2V" value="12K" x="5.08" y="16.51" rot="R90"/>
 <element name="C3" library="rcl" package="E2,5-6E" value="" x="8.89" y="7.62"/>
@@
 <wire x1="10.16" y1="7.62" x2="10.16" y2="2.54" width="0.4064" layer="16"/>
 <wire x1="10.16" y1="7.62" x2="12.7" y2="7.62" width="0.4064" layer="16"/>
-<wire x1="10.16" y1="12.7" x2="12.7" y2="12.7" width="0.4064" layer="16"/>
 <via x="12.7" y="7.62" extent="1-16" drill="0.6"/>
 <via x="12.7" y="12.7" extent="1-16" drill="0.6"/>
-<wire x1="12.7" y1="12.7" x2="12.7" y2="7.62" width="0.4064" layer="1"/>
-<wire x1="10.16" y1="12.7" x2="10.16" y2="15.24" width="0.4064" layer="16"/>
-<wire x1="10.16" y1="15.24" x2="7.62" y2="15.24" width="0.4064" layer="16"/>
-<wire x1="7.62" y1="15.24" x2="7.62" y2="20.32" width="0.4064" layer="16"/>
+<via x="7.62" y="17.78" extent="1-16" drill="0.6"/>
+<wire x1="7.62" y1="17.78" x2="7.62" y2="20.32" width="0.4064" layer="16"/>
+<wire x1="12.7" y1="7.62" x2="12.7" y2="15.24" width="0.4064" layer="16"/>
+<via x="12.7" y="15.24" extent="1-16" drill="0.6"/>
+<wire x1="12.7" y1="15.24" x2="7.62" y2="17.78" width="0.4064" layer="1"/>
+<wire x1="12.7" y1="15.24" x2="12.7" y2="12.7" width="0" layer="19" extent="1-1"/>
+<wire x1="12.7" y1="12.7" x2="10.16" y2="12.7" width="0.4064" layer="1"/>
 </signal>
 <signal name="N$10">
