File: EAGLE/ADDON/230V2LED.sch (EAGLE design)
At the start: 10 parts

Commit message: move 230V2LED -> addon dir
Parts:
- R5: value (none) -> 22K
Changed lines of the file:
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@@
 <?xml version="1.0" encoding="utf-8"?>
 <!DOCTYPE eagle SYSTEM "eagle.dtd">
-<eagle version="6.2">
+<eagle version="6.3">
 <drawing>
 <settings>
@@
 <part name="R2" library="resistor" deviceset="R-EU_" device="0207/2V" value="22K"/>
 <part name="JP2" library="pinhead" deviceset="PINHD-1X5" device=""/>
-<part name="R5" library="resistor" deviceset="R-EU_" device="0207/2V"/>
+<part name="R5" library="resistor" deviceset="R-EU_" device="0207/2V" value="22K"/>
 <part name="R1" library="resistor" deviceset="R-EU_" device="0207/2V" value="12K"/>
 <part name="C3" library="rcl" deviceset="CPOL-EU" device="E2,5-6E"/>
