File: EAGLE/ADDON/DigitalInput.brd (EAGLE design)
At the start: 15.2 x 35.6 mm, 7 parts

Commit message: update DigitalInput eagle file
Parts:
- R2: value (none) -> 10K
Changed lines of the file:
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@@
 <element name="R1" library="resistor" package="0204/7" value="" x="6.35" y="15.24" rot="R180"/>
 <element name="D2" library="diode" package="DO34Z7" value="BZV10" x="12.7" y="19.05" rot="R90"/>
-<element name="R2" library="resistor" package="0207/5V" value="" x="5.08" y="33.02" rot="R180"/>
+<element name="R2" library="resistor" package="0207/5V" value="10K" x="5.08" y="33.02" rot="R180"/>
 </elements>
 <signals>

Commit message: update eagle files
Connections:
- net N$1 renamed +5V
Changed lines of the file:
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@@
 <?xml version="1.0" encoding="utf-8"?>
 <!DOCTYPE eagle SYSTEM "eagle.dtd">
-<eagle version="6.5.0">
+<eagle version="6.6.0">
 <drawing>
 <settings>
@@
 <wire x1="12.7" y1="15.24" x2="10.16" y2="15.24" width="0.4064" layer="16"/>
 </signal>
-<signal name="N$1">
-<contactref element="OK2" pad="8"/>
-<contactref element="JP2" pad="1"/>
-<wire x1="2.54" y1="27.94" x2="2.54" y2="30.48" width="0.4064" layer="16"/>
-<wire x1="2.54" y1="33.02" x2="2.54" y2="30.48" width="0.4064" layer="16"/>
-<contactref element="R2" pad="2"/>
-<wire x1="2.54" y1="33.02" x2="2.54" y2="27.94" width="0" layer="19" extent="1-1"/>
-</signal>
 <signal name="N$3">
 <contactref element="JP2" pad="3"/>
@@
 <wire x1="2.54" y1="17.78" x2="2.54" y2="15.24" width="0.4064" layer="16"/>
 </signal>
+<signal name="+5V">
+<contactref element="OK2" pad="8"/>
+<contactref element="JP2" pad="1"/>
+<contactref element="R2" pad="2"/>
+<wire x1="2.54" y1="27.94" x2="2.54" y2="30.48" width="0.4064" layer="16"/>
+<wire x1="2.54" y1="33.02" x2="2.54" y2="30.48" width="0.4064" layer="16"/>
+</signal>
 </signals>
