File: EAGLE/ADDON/DigitalInput.sch (EAGLE design)
At the start: 7 parts

Commit message: update DigitalInput eagle file
Parts:
- R2: value (none) -> 10K
Changed lines of the file:
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@@
 <part name="R1" library="resistor" deviceset="R-EU_" device="0204/7"/>
 <part name="D2" library="diode" deviceset="BZV10" device=""/>
-<part name="R2" library="resistor" deviceset="R-EU_" device="0207/5V"/>
+<part name="R2" library="resistor" deviceset="R-EU_" device="0207/5V" value="10K"/>
 </parts>
 <sheets>

Commit message: update eagle files
Connections:
- net N$1 renamed +5V
Changed lines of the file:
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@@
 <?xml version="1.0" encoding="utf-8"?>
 <!DOCTYPE eagle SYSTEM "eagle.dtd">
-<eagle version="6.5.0">
+<eagle version="6.6.0">
 <drawing>
 <settings>
@@
 <part name="D2" library="diode" deviceset="BZV10" device=""/>
 <part name="R2" library="resistor" deviceset="R-EU_" device="0207/5V" value="10K"/>
+<part name="P+1" library="supply1" deviceset="+5V" device=""/>
 </parts>
 <sheets>
@@
 <instance part="D2" gate="1" x="-43.18" y="86.36" rot="R90"/>
 <instance part="R2" gate="G$1" x="12.7" y="88.9" rot="R90"/>
+<instance part="P+1" gate="1" x="17.78" y="101.6"/>
 </instances>
 <busses>
@@
 <pinref part="D2" gate="1" pin="C"/>
 <junction x="-43.18" y="88.9"/>
-</segment>
-</net>
-<net name="N$1" class="0">
-<segment>
-<pinref part="OK2" gate="G$1" pin="VCC"/>
-<wire x1="2.54" y1="88.9" x2="7.62" y2="88.9" width="0.1524" layer="91"/>
-<wire x1="7.62" y1="88.9" x2="7.62" y2="93.98" width="0.1524" layer="91"/>
-<wire x1="7.62" y1="93.98" x2="12.7" y2="93.98" width="0.1524" layer="91"/>
-<wire x1="12.7" y1="93.98" x2="20.32" y2="93.98" width="0.1524" layer="91"/>
-<wire x1="20.32" y1="93.98" x2="20.32" y2="88.9" width="0.1524" layer="91"/>
-<pinref part="JP2" gate="A" pin="1"/>
-<wire x1="20.32" y1="88.9" x2="25.4" y2="88.9" width="0.1524" layer="91"/>
-<pinref part="R2" gate="G$1" pin="2"/>
-<junction x="12.7" y="93.98"/>
 </segment>
 </net>
@@
 </segment>
 </net>
+<net name="+5V" class="0">
+<segment>
+<pinref part="OK2" gate="G$1" pin="VCC"/>
+<wire x1="2.54" y1="88.9" x2="7.62" y2="88.9" width="0.1524" layer="91"/>
+<wire x1="7.62" y1="88.9" x2="7.62" y2="93.98" width="0.1524" layer="91"/>
+<wire x1="7.62" y1="93.98" x2="12.7" y2="93.98" width="0.1524" layer="91"/>
+<wire x1="12.7" y1="93.98" x2="17.78" y2="93.98" width="0.1524" layer="91"/>
+<wire x1="17.78" y1="93.98" x2="20.32" y2="93.98" width="0.1524" layer="91"/>
+<wire x1="20.32" y1="93.98" x2="20.32" y2="88.9" width="0.1524" layer="91"/>
+<pinref part="JP2" gate="A" pin="1"/>
+<wire x1="20.32" y1="88.9" x2="25.4" y2="88.9" width="0.1524" layer="91"/>
+<pinref part="R2" gate="G$1" pin="2"/>
+<junction x="12.7" y="93.98"/>
+<pinref part="P+1" gate="1" pin="+5V"/>
+<wire x1="17.78" y1="93.98" x2="17.78" y2="99.06" width="0.1524" layer="91"/>
+</segment>
+</net>
