File: EAGLE/AVRI2CIO_V0_2_TOPLEVEL.brd (EAGLE design)
At the start: 99.1 x 40.6 mm, 3 parts, among them IC1 MEGA8-P

Commit message: update eagle files
Connections:
- new net N$1: JP1.1
- net PB1: no longer JP1.1
Routing:
- net PB1: track 43.2 -> 0.00 mm
Changed lines of the file:
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@@
 <?xml version="1.0" encoding="utf-8"?>
 <!DOCTYPE eagle SYSTEM "eagle.dtd">
-<eagle version="6.3">
+<eagle version="6.5.0">
 <drawing>
 <settings>
@@
 <contactref element="JP1" pad="8"/>
 <contactref element="JP2" pad="8"/>
-<wire x1="45.72" y1="27.94" x2="53.34" y2="30.48" width="0" layer="19" extent="1-1"/>
 <wire x1="2.54" y1="27.94" x2="45.72" y2="27.94" width="0.4064" layer="16"/>
 <wire x1="96.52" y1="30.48" x2="53.34" y2="30.48" width="0.4064" layer="16"/>
+<wire x1="45.72" y1="27.94" x2="53.34" y2="30.48" width="0" layer="19" extent="1-1"/>
 </signal>
 <signal name="+5V">
@@
 <signal name="PB1">
 <contactref element="IC1" pad="15"/>
-<contactref element="JP1" pad="1"/>
-<wire x1="2.54" y1="45.72" x2="45.72" y2="45.72" width="0.4064" layer="16"/>
 </signal>
 <signal name="PB4">
@@
 <wire x1="96.52" y1="25.4" x2="53.34" y2="25.4" width="0.4064" layer="16"/>
 </signal>
+<signal name="N$1">
+<contactref element="JP1" pad="1"/>
+</signal>
 </signals>
