File: EAGLE/AVRI2CIO_V0_2_TOPLEVEL.sch (EAGLE design)
At the start: 3 parts, among them IC1 MEGA8-P

Commit message: update eagle files
Connections:
- new net N$1: JP1.1
- net PB1: no longer JP1.1
Changed lines of the file:
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@@
 <?xml version="1.0" encoding="utf-8"?>
 <!DOCTYPE eagle SYSTEM "eagle.dtd">
-<eagle version="6.3">
+<eagle version="6.5.0">
 <drawing>
 <settings>
@@
 <label x="154.94" y="-170.18" size="1.778" layer="95"/>
 </segment>
-<segment>
-<wire x1="25.4" y1="-124.46" x2="35.56" y2="-124.46" width="0.1524" layer="91"/>
-<label x="38.1" y="-124.46" size="1.778" layer="95"/>
-<pinref part="JP1" gate="A" pin="1"/>
-</segment>
 </net>
 <net name="PB4" class="0">
@@
 </segment>
 </net>
+<net name="N$1" class="0">
+<segment>
+<pinref part="JP1" gate="A" pin="1"/>
+<wire x1="25.4" y1="-124.46" x2="35.56" y2="-124.46" width="0.1524" layer="91"/>
+<label x="38.1" y="-124.46" size="1.778" layer="95"/>
+</segment>
+</net>
