File: EAGLE/AVRI2CIO.brd (EAGLE design)
At the start: 99.1 x 78.7 mm, 39 parts, among them IC1 MEGA8-P

Commit message: update eagle files
Parts:
- removed PH0_E: (no value), pinhead:1X03
- added JP1, JP2: (no value), pinhead:1X06
Connections:
- removed net N$1: PH0_E.3, X10.2
- removed net N$17: PH0_E.1, X10.1
- removed net SCL: IC1.28, X9.2
- removed net SDA: IC1.27, X9.1
- new net GND_LL: JP1.3, X9.2
- new net SCL_HL: IC1.28, JP2.1
- new net SCL_LL: JP1.6, X10.2
- new net SDA_HL: IC1.27, JP2.6
- new net SDA_LL: JP1.1, X9.1
- new net VCC_LL: JP1.4, X10.1
- net +5V: now also JP2.4
- net GND: now also JP2.3
Routing:
- net SDA: track 71.2 -> 0.00 mm, vias 4 -> 0
- net SCL: track 68.5 -> 0.00 mm, vias 4 -> 0
- net SCL_HL: track 0.00 -> 50.8 mm, vias 0 -> 2
- net SDA_HL: track 0.00 -> 45.7 mm, vias 0 -> 2
- net N$1: track 25.4 -> 0.00 mm
- net +5V: track 361.3 -> 376.6 mm
- net GND: track 225.4 -> 240.7 mm
- net SDA_LL: track 0.00 -> 12.7 mm
- net GND_LL: track 0.00 -> 12.7 mm
- net VCC_LL: track 0.00 -> 10.2 mm
- net SCL_LL: track 0.00 -> 10.2 mm
- net N$17: track 5.08 -> 0.00 mm
Changed lines of the file:
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@@
 <?xml version="1.0" encoding="utf-8"?>
 <!DOCTYPE eagle SYSTEM "eagle.dtd">
-<eagle version="6.2">
+<eagle version="6.3">
 <drawing>
 <settings>
@@
 </class>
 </classes>
-<designrules>
+<designrules name="default">
 <description language="de">&lt;b&gt;EAGLE Design Rules&lt;/b&gt;
 &lt;p&gt;
@@
 <attribute name="VALUE" x="92.71" y="10.795" size="1.27" layer="27" rot="R180"/>
 </element>
-<element name="PH0_E" library="pinhead" package="1X03" value="" x="12.7" y="71.12" rot="R180"/>
 <element name="PH1_E" library="pinhead" package="1X03" value="" x="27.94" y="71.12" smashed="yes">
 <attribute name="NAME" x="24.0538" y="67.8688" size="1.27" layer="25" ratio="10"/>
@@
 <attribute name="OC_FARNELL" value="unknown" x="7.62" y="77.47" size="1.778" layer="27" display="off"/>
 </element>
+<element name="JP1" library="pinhead" package="1X06" value="" x="13.97" y="66.04"/>
+<element name="JP2" library="pinhead" package="1X06" value="" x="13.97" y="55.88"/>
 </elements>
 <signals>
@@
 <via x="76.2" y="45.72" extent="1-16" drill="0.6"/>
 <wire x1="76.2" y1="45.72" x2="76.2" y2="43.18" width="0.4064" layer="16"/>
+<contactref element="JP2" pad="3"/>
+<wire x1="10.16" y1="43.18" x2="10.16" y2="53.34" width="0.4064" layer="16"/>
+<wire x1="12.7" y1="55.88" x2="12.7" y2="53.34" width="0.4064" layer="16"/>
+<wire x1="12.7" y1="53.34" x2="10.16" y2="53.34" width="0.4064" layer="16"/>
 </signal>
 <signal name="+5V">
@@
 <wire x1="2.54" y1="2.54" x2="2.54" y2="7.62" width="0.4064" layer="16"/>
 <wire x1="68.58" y1="53.34" x2="68.58" y2="43.18" width="0.4064" layer="16"/>
+<contactref element="JP2" pad="4"/>
+<wire x1="17.78" y1="43.18" x2="17.78" y2="53.34" width="0.4064" layer="16"/>
+<wire x1="17.78" y1="53.34" x2="15.24" y2="53.34" width="0.4064" layer="16"/>
+<wire x1="15.24" y1="53.34" x2="15.24" y2="55.88" width="0.4064" layer="16"/>
 </signal>
 <signal name="IO1">
 <contactref element="IC1" pad="9"/>
 </signal>
-<signal name="SDA">
+<signal name="SDA_HL">
 <contactref element="IC1" pad="27"/>
-<contactref element="X9" pad="1"/>
-<wire x1="55.88" y1="60.96" x2="55.88" y2="63.5" width="0.4064" layer="16"/>
+<contactref element="JP2" pad="6"/>
+<wire x1="20.32" y1="55.88" x2="20.32" y2="63.5" width="0.4064" layer="16"/>
+<via x="20.32" y="63.5" extent="1-16" drill="0.6"/>
+<wire x1="20.32" y1="63.5" x2="55.88" y2="63.5" width="0.4064" layer="1"/>
 <via x="55.88" y="63.5" extent="1-16" drill="0.6"/>
-<wire x1="55.88" y1="63.5" x2="7.62" y2="63.5" width="0.4064" layer="1"/>
-<via x="7.62" y="63.5" extent="1-16" drill="0.6"/>
-<wire x1="7.62" y1="63.5" x2="2.54" y2="63.5" width="0.4064" layer="16"/>
-<wire x1="5.12" y1="76.2" x2="2.54" y2="76.2" width="0.4064" layer="16"/>
-<via x="2.54" y="63.5" extent="1-16" drill="0.6"/>
-<via x="2.54" y="76.2" extent="1-16" drill="0.6"/>
-<wire x1="2.54" y1="76.2" x2="2.54" y2="63.5" width="0.4064" layer="1"/>
-</signal>
-<signal name="SCL">
+<wire x1="55.88" y1="63.5" x2="55.88" y2="60.96" width="0.4064" layer="16"/>
+</signal>
+<signal name="SCL_HL">
 <contactref element="IC1" pad="28"/>
-<contactref element="X9" pad="2"/>
-<wire x1="10.12" y1="76.2" x2="7.62" y2="76.2" width="0.4064" layer="16"/>
-<wire x1="7.62" y1="76.2" x2="7.62" y2="73.66" width="0.4064" layer="16"/>
-<wire x1="7.62" y1="73.66" x2="5.08" y2="73.66" width="0.4064" layer="16"/>
-<wire x1="5.08" y1="73.66" x2="5.08" y2="68.58" width="0.4064" layer="16"/>
-<via x="5.08" y="68.58" extent="1-16" drill="0.6"/>
-<wire x1="5.08" y1="68.58" x2="5.08" y2="60.96" width="0.4064" layer="1"/>
-<via x="5.08" y="60.96" extent="1-16" drill="0.6"/>
-<wire x1="5.08" y1="60.96" x2="7.62" y2="60.96" width="0.4064" layer="16"/>
-<via x="7.62" y="60.96" extent="1-16" drill="0.6"/>
-<wire x1="7.62" y1="60.96" x2="50.8" y2="60.96" width="0.4064" layer="1"/>
+<wire x1="53.34" y1="60.96" x2="50.8" y2="60.96" width="0.4064" layer="16"/>
 <via x="50.8" y="60.96" extent="1-16" drill="0.6"/>
-<wire x1="50.8" y1="60.96" x2="53.34" y2="60.96" width="0.4064" layer="16"/>
+<wire x1="50.8" y1="60.96" x2="7.62" y2="60.96" width="0.4064" layer="1"/>
+<via x="7.62" y="60.96" extent="1-16" drill="0.6" shape="square"/>
+<contactref element="JP2" pad="1"/>
+<wire x1="7.62" y1="55.88" x2="7.62" y2="60.96" width="0.4064" layer="16"/>
 </signal>
 <signal name="IO13">
@@
 <wire x1="45.72" y1="58.42" x2="45.72" y2="66.04" width="0.4064" layer="16"/>
 </signal>
-<signal name="N$1">
-<contactref element="PH0_E" pad="3"/>
+<signal name="VCC_LL">
+<contactref element="X10" pad="1"/>
+<contactref element="JP1" pad="4"/>
+<wire x1="15.24" y1="66.04" x2="15.28" y2="76.2" width="0" layer="19" extent="1-1"/>
+<wire x1="15.24" y1="76.2" x2="15.24" y2="66.04" width="0.4064" layer="16"/>
+</signal>
+<signal name="SDA_LL">
+<contactref element="X9" pad="1"/>
+<wire x1="5.12" y1="76.2" x2="5.08" y2="76.2" width="0.4064" layer="16"/>
+<wire x1="5.08" y1="76.2" x2="5.08" y2="66.04" width="0.4064" layer="16"/>
+<contactref element="JP1" pad="1"/>
+<wire x1="5.08" y1="66.04" x2="7.62" y2="66.04" width="0.4064" layer="16"/>
+</signal>
+<signal name="SCL_LL">
 <contactref element="X10" pad="2"/>
-<wire x1="10.16" y1="71.12" x2="10.16" y2="66.04" width="0.4064" layer="16"/>
-<wire x1="20.32" y1="66.04" x2="20.28" y2="76.2" width="0.4064" layer="16"/>
-<wire x1="10.16" y1="66.04" x2="20.32" y2="66.04" width="0.4064" layer="16"/>
-</signal>
-<signal name="N$17">
-<contactref element="PH0_E" pad="1"/>
-<contactref element="X10" pad="1"/>
-<wire x1="15.28" y1="76.2" x2="15.24" y2="71.12" width="0.4064" layer="16"/>
+<contactref element="JP1" pad="6"/>
+<wire x1="20.32" y1="66.04" x2="20.28" y2="76.2" width="0" layer="19" extent="1-1"/>
+<wire x1="20.32" y1="76.2" x2="20.32" y2="66.04" width="0.4064" layer="16"/>
+</signal>
+<signal name="GND_LL">
+<contactref element="X9" pad="2"/>
+<contactref element="JP1" pad="3"/>
+<wire x1="10.12" y1="76.2" x2="10.12" y2="71.16" width="0.4064" layer="16"/>
+<wire x1="10.12" y1="71.16" x2="10.16" y2="71.12" width="0.4064" layer="16"/>
+<wire x1="10.16" y1="71.12" x2="12.7" y2="71.12" width="0.4064" layer="16"/>
+<wire x1="12.7" y1="71.12" x2="12.7" y2="66.04" width="0.4064" layer="16"/>
 </signal>
 </signals>
