File: EAGLE/AVRI2CIO.sch (EAGLE design)
At the start: 39 parts, among them IC1 MEGA8-P

Commit message: update eagle files
Parts:
- removed PH0_E: (no value), pinhead:PINHD-1X3
- added JP1, JP2: (no value), pinhead:PINHD-1X6
Connections:
- removed net N$1: PH0_E.3, X10-2.KL
- removed net N$17: PH0_E.1, X10-1.KL
- removed net SCL: IC1.PC5(ADC5/SCL), X9-2.KL
- removed net SDA: IC1.PC4(ADC4/SDA), X9-1.KL
- new net GND_LL: JP1.3, X9-2.KL
- new net SCL_HL: IC1.PC5(ADC5/SCL), JP2.1
- new net SCL_LL: JP1.6, X10-2.KL
- new net SDA_HL: IC1.PC4(ADC4/SDA), JP2.6
- new net SDA_LL: JP1.1, X9-1.KL
- new net VCC_LL: JP1.4, X10-1.KL
- net +5V: now also JP2.4
- net GND: now also JP2.3
Other:
- moved on the sheet: X10-1, X10-2, X9-1, X9-2
Changed lines of the file:
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@@
 <?xml version="1.0" encoding="utf-8"?>
 <!DOCTYPE eagle SYSTEM "eagle.dtd">
-<eagle version="6.2">
+<eagle version="6.3">
 <drawing>
 <settings>
@@
 <part name="PH10_E" library="pinhead" deviceset="PINHD-1X3" device=""/>
 <part name="PH11_E" library="pinhead" deviceset="PINHD-1X3" device=""/>
-<part name="PH0_E" library="pinhead" deviceset="PINHD-1X3" device=""/>
 <part name="PH1_E" library="pinhead" deviceset="PINHD-1X3" device=""/>
 <part name="PH2_E" library="pinhead" deviceset="PINHD-1X3" device=""/>
@@
 <part name="GND25" library="supply1" deviceset="GND" device=""/>
 <part name="X9" library="con-wago-500" deviceset="W237-102" device=""/>
+<part name="JP1" library="pinhead" deviceset="PINHD-1X6" device=""/>
+<part name="JP2" library="pinhead" deviceset="PINHD-1X6" device=""/>
 </parts>
 <sheets>
@@
 <instance part="PH10_E" gate="A" x="170.18" y="-185.42" rot="R90"/>
 <instance part="PH11_E" gate="A" x="195.58" y="-185.42" rot="R90"/>
-<instance part="PH0_E" gate="A" x="68.58" y="-111.76" rot="R270"/>
 <instance part="PH1_E" gate="A" x="93.98" y="-111.76" rot="R270"/>
 <instance part="PH2_E" gate="A" x="119.38" y="-111.76" rot="R270"/>
@@
 <instance part="PH4_E" gate="A" x="170.18" y="-111.76" rot="R270"/>
 <instance part="PH5_E" gate="A" x="195.58" y="-111.76" rot="R270"/>
-<instance part="X10" gate="-1" x="71.12" y="-96.52" rot="R270"/>
-<instance part="X10" gate="-2" x="66.04" y="-96.52" rot="R270"/>
+<instance part="X10" gate="-1" x="-7.62" y="-127" rot="R180"/>
+<instance part="X10" gate="-2" x="-7.62" y="-121.92" rot="R180"/>
 <instance part="X11" gate="-1" x="96.52" y="-96.52" rot="R270"/>
 <instance part="X11" gate="-2" x="91.44" y="-96.52" rot="R270"/>
@@
 <instance part="GND24" gate="1" x="147.32" y="-139.7"/>
 <instance part="GND25" gate="1" x="172.72" y="-139.7"/>
-<instance part="X9" gate="-1" x="-35.56" y="71.12"/>
-<instance part="X9" gate="-2" x="-35.56" y="66.04"/>
+<instance part="X9" gate="-1" x="-7.62" y="-134.62" rot="R180"/>
+<instance part="X9" gate="-2" x="-7.62" y="-129.54" rot="R180"/>
+<instance part="JP1" gate="A" x="-33.02" y="-127" rot="R180"/>
+<instance part="JP2" gate="A" x="10.16" y="-127" rot="R180"/>
 </instances>
 <busses>
@@
 <junction x="-15.24" y="48.26"/>
 </segment>
+<segment>
+<pinref part="JP2" gate="A" pin="3"/>
+<wire x1="12.7" y1="-129.54" x2="25.4" y2="-129.54" width="0.1524" layer="91"/>
+<label x="27.94" y="-129.54" size="1.778" layer="95"/>
+</segment>
 </net>
 <net name="+5V" class="0">
@@
 <wire x1="200.66" y1="-165.1" x2="200.66" y2="-172.72" width="0.1524" layer="91"/>
 </segment>
+<segment>
+<pinref part="JP2" gate="A" pin="4"/>
+<wire x1="12.7" y1="-127" x2="25.4" y2="-127" width="0.1524" layer="91"/>
+<label x="27.94" y="-127" size="1.778" layer="95"/>
+</segment>
 </net>
 <net name="IO1" class="0">
@@
 </segment>
 </net>
-<net name="SDA" class="0">
+<net name="SDA_HL" class="0">
 <segment>
 <pinref part="IC1" gate="G$1" pin="PC4(ADC4/SDA)"/>
 <wire x1="43.18" y1="68.58" x2="53.34" y2="68.58" width="0.1524" layer="91"/>
-<label x="45.72" y="68.58" size="1.778" layer="95"/>
-</segment>
-<segment>
-<pinref part="X9" gate="-1" pin="KL"/>
-<wire x1="-30.48" y1="71.12" x2="-22.86" y2="71.12" width="0.1524" layer="91"/>
-<label x="-22.86" y="71.12" size="1.778" layer="95"/>
-</segment>
-</net>
-<net name="SCL" class="0">
+<label x="58.42" y="68.58" size="1.778" layer="95"/>
+</segment>
+<segment>
+<pinref part="JP2" gate="A" pin="6"/>
+<wire x1="12.7" y1="-121.92" x2="25.4" y2="-121.92" width="0.1524" layer="91"/>
+<label x="20.32" y="-121.92" size="1.778" layer="95"/>
+</segment>
+</net>
+<net name="SCL_HL" class="0">
 <segment>
 <pinref part="IC1" gate="G$1" pin="PC5(ADC5/SCL)"/>
 <wire x1="43.18" y1="66.04" x2="53.34" y2="66.04" width="0.1524" layer="91"/>
-<label x="45.72" y="66.04" size="1.778" layer="95"/>
-</segment>
-<segment>
-<pinref part="X9" gate="-2" pin="KL"/>
-<wire x1="-30.48" y1="66.04" x2="-22.86" y2="66.04" width="0.1524" layer="91"/>
-<label x="-22.86" y="66.04" size="1.778" layer="95"/>
+<label x="58.42" y="66.04" size="1.778" layer="95"/>
+</segment>
+<segment>
+<pinref part="JP2" gate="A" pin="1"/>
+<wire x1="12.7" y1="-134.62" x2="25.4" y2="-134.62" width="0.1524" layer="91"/>
+<label x="20.32" y="-134.62" size="1.778" layer="95"/>
 </segment>
 </net>
@@
 <pinref part="IC1" gate="G$1" pin="PC3(ADC3)"/>
 <wire x1="43.18" y1="71.12" x2="53.34" y2="71.12" width="0.1524" layer="91"/>
-<label x="45.72" y="71.12" size="1.778" layer="95"/>
+<label x="58.42" y="71.12" size="1.778" layer="95"/>
 </segment>
 <segment>
@@
 </segment>
 </net>
-<net name="N$1" class="0">
-<segment>
-<pinref part="PH0_E" gate="A" pin="3"/>
+<net name="VCC_LL" class="0">
+<segment>
+<pinref part="X10" gate="-1" pin="KL"/>
+<pinref part="JP1" gate="A" pin="4"/>
+<wire x1="-12.7" y1="-127" x2="-30.48" y2="-127" width="0.1524" layer="91"/>
+<label x="-22.86" y="-127" size="1.778" layer="95"/>
+</segment>
+</net>
+<net name="SDA_LL" class="0">
+<segment>
+<pinref part="X9" gate="-1" pin="KL"/>
+<pinref part="JP1" gate="A" pin="1"/>
+<wire x1="-30.48" y1="-134.62" x2="-12.7" y2="-134.62" width="0.1524" layer="91"/>
+<label x="-22.86" y="-134.62" size="1.778" layer="95"/>
+</segment>
+</net>
+<net name="SCL_LL" class="0">
+<segment>
 <pinref part="X10" gate="-2" pin="KL"/>
-<wire x1="66.04" y1="-109.22" x2="66.04" y2="-101.6" width="0.1524" layer="91"/>
-</segment>
-</net>
-<net name="N$17" class="0">
-<segment>
-<pinref part="PH0_E" gate="A" pin="1"/>
-<pinref part="X10" gate="-1" pin="KL"/>
-<wire x1="71.12" y1="-109.22" x2="71.12" y2="-101.6" width="0.1524" layer="91"/>
-</segment>
-</net>
+<wire x1="-12.7" y1="-121.92" x2="-30.48" y2="-121.92" width="0.1524" layer="91"/>
+<pinref part="JP1" gate="A" pin="6"/>
+<label x="-22.86" y="-121.92" size="1.778" layer="95"/>
+</segment>
+</net>
+<net name="GND_LL" class="0">
+<segment>
+<pinref part="X9" gate="-2" pin="KL"/>
+<wire x1="-12.7" y1="-129.54" x2="-30.48" y2="-129.54" width="0.1524" layer="91"/>
+<pinref part="JP1" gate="A" pin="3"/>
+<label x="-22.86" y="-129.54" size="1.778" layer="95"/>
+</segment>
+</net>
