File: EAGLE/AVRI2CIO_V0_2_LEVEL0.brd (EAGLE design)
At the start: 99.1 x 78.7 mm, 38 parts

Commit message: update eagle files
Connections:
- net N$22: now also JP3.13; no longer JP3.1
Routing:
- net N$22: track 99.5 -> 132.1 mm, vias 4 -> 3
Changed lines of the file:
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@@
 <?xml version="1.0" encoding="utf-8"?>
 <!DOCTYPE eagle SYSTEM "eagle.dtd">
-<eagle version="6.3">
+<eagle version="6.5.0">
 <drawing>
 <settings>
@@
 <wire x1="27.94" y1="22.86" x2="27.94" y2="35.56" width="0.4064" layer="16"/>
 </signal>
-<signal name="N$22">
-<contactref element="PH6_I" pad="3"/>
-<contactref element="JP3" pad="1"/>
-<wire x1="96.52" y1="22.86" x2="93.98" y2="22.86" width="0.4064" layer="16"/>
-<via x="93.98" y="22.86" extent="1-16" drill="0.6"/>
-<wire x1="12.7" y1="35.56" x2="12.7" y2="20.32" width="0.4064" layer="16"/>
-<via x="12.7" y="20.32" extent="1-16" drill="0.6"/>
-<wire x1="12.7" y1="20.32" x2="83.82" y2="20.32" width="0.4064" layer="1"/>
-<via x="83.82" y="20.32" extent="1-16" drill="0.6"/>
-<wire x1="83.82" y1="20.32" x2="86.36" y2="20.32" width="0.4064" layer="16"/>
-<via x="86.36" y="20.32" extent="1-16" drill="0.6"/>
-<wire x1="86.36" y1="20.32" x2="93.98" y2="22.86" width="0.4064" layer="1"/>
-</signal>
 <signal name="N$31">
 <contactref element="PH11_I" pad="3"/>
@@
 <via x="93.98" y="25.4" extent="1-16" drill="0.6"/>
 </signal>
+<signal name="N$62">
+<via x="93.98" y="53.34" extent="1-16" drill="0.6"/>
+</signal>
+<signal name="N$63">
+<via x="66.04" y="53.34" extent="1-16" drill="0.6"/>
+</signal>
+<signal name="N$22">
+<contactref element="PH6_I" pad="3"/>
+<contactref element="JP3" pad="13"/>
+<wire x1="96.52" y1="53.34" x2="93.98" y2="53.34" width="0.4064" layer="16"/>
+<wire x1="12.7" y1="35.56" x2="12.7" y2="20.32" width="0.4064" layer="16"/>
+<via x="12.7" y="20.32" extent="1-16" drill="0.6"/>
+<wire x1="12.7" y1="20.32" x2="66.04" y2="20.32" width="0.4064" layer="1"/>
+<via x="66.04" y="20.32" extent="1-16" drill="0.6"/>
+<wire x1="66.04" y1="20.32" x2="66.04" y2="53.34" width="0.4064" layer="16"/>
+<via x="66.04" y="53.34" extent="1-16" drill="0.6"/>
+<wire x1="66.04" y1="53.34" x2="93.98" y2="53.34" width="0.4064" layer="1"/>
+<wire x1="93.98" y1="53.34" x2="93.98" y2="53.34" width="0" layer="19" extent="1-16"/>
+</signal>
+<signal name="N$64">
+<via x="66.04" y="20.32" extent="1-16" drill="0.6"/>
+</signal>
 </signals>

Commit message: update eagle files
Parts:
- added DRILEGEND: (no value), drilegend:DRILEGEND
Connections:
- removed net N$37: JP4.11
- net N$16: now also JP4.12, PH7_I.3; no longer JP4.2, PH3_I.3
- net N$18: now also PH9_I.3; no longer PH8_I.3
- net N$21: now also PH8_I.3; no longer PH7_I.3
- net N$22: now also PH3_I.3; no longer PH6_I.3
- net N$31: now also PH4_I.3; no longer PH11_I.3
- net N$32: now also PH1_I.3; no longer PH2_I.3
- net N$34: now also JP4.11, PH6_I.3; no longer JP4.4, PH1_I.3
- net N$36: now also PH2_I.3; no longer PH4_I.3
- net PD3: now also PH10_I.3; no longer PH9_I.3
- net PD5: now also PH11_I.3; no longer PH10_I.3
Routing:
- net N$22: track 132.1 -> 48.3 mm, vias 3 -> 0
- net N$31: track 73.7 -> 30.5 mm, vias 5 -> 0
- net GND: track 251.5 -> 213.4 mm, vias 24 -> 0
- net N$16: track 66.0 -> 33.0 mm, vias 2 -> 0
- net N$36: track 83.8 -> 53.3 mm, vias 2 -> 0
- net PD5: track 28.4 -> 10.2 mm, vias 4 -> 0
- net N$21: track 81.7 -> 63.5 mm, vias 4 -> 0
- net N$18: track 63.9 -> 45.7 mm, vias 3 -> 0
- net PD3: track 46.1 -> 27.9 mm, vias 4 -> 0
- net N$32: track 48.3 -> 33.0 mm, vias 2 -> 0
- net N$34: track 30.5 -> 15.2 mm, vias 2 -> 0
- net N$4: track 0.00 -> 5.08 mm
- net N$2: track 0.00 -> 5.08 mm
- net N$1: track 0.00 -> 5.08 mm
- net N$17: track 10.8 -> 12.7 mm, vias 2 -> 0
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Other:
- board text added: "01-16"
- board text added: "01-20"
- board text added: "LAYER-STACK"
