File: EAGLE/AVRI2CIO_V0_2_LEVEL0.sch (EAGLE design)
At the start: 38 parts

Commit message: update eagle files
Connections:
- net N$22: now also JP3.13; no longer JP3.1
Changed lines of the file:
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@@
 <?xml version="1.0" encoding="utf-8"?>
 <!DOCTYPE eagle SYSTEM "eagle.dtd">
-<eagle version="6.3">
+<eagle version="6.5.0">
 <drawing>
 <settings>
@@
 </segment>
 </net>
-<net name="N$22" class="0">
-<segment>
-<pinref part="PH6_I" gate="A" pin="3"/>
-<wire x1="119.38" y1="-160.02" x2="119.38" y2="-195.58" width="0.1524" layer="91"/>
-<pinref part="JP3" gate="A" pin="1"/>
-<wire x1="119.38" y1="-160.02" x2="246.38" y2="-160.02" width="0.1524" layer="91"/>
-</segment>
-</net>
 <net name="N$31" class="0">
 <segment>
@@
 </segment>
 </net>
+<net name="N$22" class="0">
+<segment>
+<pinref part="PH6_I" gate="A" pin="3"/>
+<wire x1="119.38" y1="-195.58" x2="119.38" y2="-144.78" width="0.1524" layer="91"/>
+<wire x1="119.38" y1="-144.78" x2="208.28" y2="-144.78" width="0.1524" layer="91"/>
+<wire x1="208.28" y1="-144.78" x2="208.28" y2="-129.54" width="0.1524" layer="91"/>
+<pinref part="JP3" gate="A" pin="13"/>
+<wire x1="208.28" y1="-129.54" x2="246.38" y2="-129.54" width="0.1524" layer="91"/>
+</segment>
+</net>

Commit message: update eagle files
Connections:
- removed net N$37: JP4.11
- net N$16: now also JP4.12, PH7_I.3; no longer JP4.2, PH3_I.3
- net N$18: now also PH9_I.3; no longer PH8_I.3
- net N$21: now also PH8_I.3; no longer PH7_I.3
- net N$22: now also PH3_I.3; no longer PH6_I.3
- net N$31: now also PH4_I.3; no longer PH11_I.3
- net N$32: now also PH1_I.3; no longer PH2_I.3
- net N$34: now also JP4.11, PH6_I.3; no longer JP4.4, PH1_I.3
- net N$36: now also PH2_I.3; no longer PH4_I.3
- net PD3: now also PH10_I.3; no longer PH9_I.3
- net PD5: now also PH11_I.3; no longer PH10_I.3
Other:
- moved on the sheet: PH2_E, PH2_I, PH6_E, PH6_I, PH7_E, PH7_I, PH8_E, PH8_I, X12-1, X12-2, X3-1, X3-2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
