File: EAGLE/AVRI2CIO_V0_2_LEVEL1.brd (EAGLE design)
At the start: 99.1 x 58.4 mm, 18 parts

Commit message: update eagle files
Parts:
- added JP5: (no value), pinhead:1X01
- added PH5_I1, PH5_I2: (no value), pinhead:1X05
- added X3, X4: (no value), con-wago-500:W237-102
- JP1: value (none) -> I2C
- moved X1 66.7 mm to (53.3, 14.0), turned to 180 degrees
- moved X2 51.1 mm to (25.4, 14.0), turned to 180 degrees
- moved X11 50.9 mm to (88.9, 64.8), turned to 0 degrees
- moved X12 50.9 mm to (73.7, 64.8), turned to 0 degrees
- moved X15 50.9 mm to (58.4, 64.8), turned to 0 degrees
- moved X10 50.8 mm to (43.2, 64.8), turned to 0 degrees
- moved PH0_I 49.1 mm to (88.9, 30.5)
- moved PH1_I 49.1 mm to (43.2, 30.5)
- moved JP1 47.9 mm to (39.4, 12.7), turned to 180 degrees
- moved PH0_E 38.1 mm to (43.2, 58.4), turned to 0 degrees
- moved PH1_E 38.1 mm to (88.9, 58.4), turned to 0 degrees
- moved PH2_E 38.1 mm to (73.7, 58.4), turned to 0 degrees
- moved PH5_E 38.1 mm to (58.4, 58.4), turned to 0 degrees
- moved JP2 32.5 mm to (39.4, 22.9), turned to 180 degrees
- moved PH2_I 23.4 mm to (58.4, 30.5)
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Connections:
- removed net N$3: JP3.11, PH2_I.3
- removed net N$4: JP3.12, PH1_I.3
- new net N$14: PH5_I1.2, X3.2
- new net N$16: PH5_I1.4, X3.1
- new net N$18: JP3.2, PH0_I.3
- new net N$22: JP3.4, PH5_I.3
- net +5V: now also PH5_I2.4, X4.2
- net GND: now also PH5_I2.2, X4.1
- net N$10: now also JP1.6, X2.1; no longer JP1.1, X1.1
- net N$11: now also JP2.1; no longer JP2.6
- net N$12: now also JP2.6; no longer JP2.1
- net N$5: now also PH1_I.3; no longer PH5_I.3
- net N$6: now also PH2_I.3; no longer PH0_I.3
- net N$7: now also JP1.1, X1.2; no longer JP1.6, X2.2
- net N$8: now also JP1.3, X1.1; no longer JP1.4, X2.1
- net N$9: now also JP1.4, X2.2; no longer JP1.3, X1.2
Routing:
- net N$18: track 0.00 -> 109.2 mm, vias 0 -> 2
- net N$4: track 106.7 -> 0.00 mm, vias 2 -> 0
- net N$3: track 88.9 -> 0.00 mm, vias 2 -> 0
- net N$22: track 0.00 -> 88.9 mm, vias 0 -> 2
- net GND: track 165.1 -> 205.8 mm, vias 19 -> 4
- net +5V: track 149.9 -> 185.5 mm, vias 18 -> 4
- net N$5: track 71.1 -> 43.2 mm
- net N$9: track 10.2 -> 22.9 mm
- net N$6: track 53.3 -> 66.0 mm
- net N$8: track 11.2 -> 22.9 mm, vias 2 -> 0
- net N$11: track 38.1 -> 49.5 mm, vias 2 -> 0
- net N$12: track 22.9 -> 33.0 mm
- net N$16: track 0.00 -> 5.12 mm
- net N$14: track 0.00 -> 5.12 mm
- net N$7: track 11.2 -> 7.62 mm, vias 2 -> 0
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- added copper zone on layer 16, net N$3
Other:
- board text removed: "I2C Pegelwandler"
