File: EAGLE/AVRI2CIO_V0_2_LEVEL1.sch (EAGLE design)
At the start: 18 parts

Commit message: update eagle files
Parts:
- added JP5: (no value), pinhead:PINHD-1X1
- added PH5_I1, PH5_I2: (no value), pinhead:PINHD-1X5
- added X3, X4: (no value), con-wago-500:W237-102
- JP1: value (none) -> I2C
Connections:
- removed net N$3: JP3.11, PH2_I.3
- removed net N$4: JP3.12, PH1_I.3
- new net N$14: PH5_I1.2, X3-2.KL
- new net N$16: PH5_I1.4, X3-1.KL
- new net N$18: JP3.2, PH0_I.3
- new net N$22: JP3.4, PH5_I.3
- net +5V: now also PH5_I2.4, X4-2.KL
- net GND: now also PH5_I2.2, X4-1.KL
- net N$10: now also JP1.6, X2-1.KL; no longer JP1.1, X1-1.KL
- net N$11: now also JP2.1; no longer JP2.6
- net N$12: now also JP2.6; no longer JP2.1
- net N$5: now also PH1_I.3; no longer PH5_I.3
- net N$6: now also PH2_I.3; no longer PH0_I.3
- net N$7: now also JP1.1, X1-2.KL; no longer JP1.6, X2-2.KL
- net N$8: now also JP1.3, X1-1.KL; no longer JP1.4, X2-1.KL
- net N$9: now also JP1.4, X2-2.KL; no longer JP1.3, X1-2.KL
Other:
- moved on the sheet: JP2, X1-1, X1-2, X2-1, X2-2
