File: EAGLE/MainBoard/V0_2/AVRI2CIO_V0_2_LEVEL0.brd (EAGLE design)
At the start: 99.1 x 78.7 mm, 39 parts

Commit message: update eagle files
Parts:
- X10, X11, X12, X13, X14, X15, X3, X4, X5, X6, X7, X8: device con-wago-500:W237-102 -> con-wago-508:W237-132
Routing:
- net N$8: track 5.08 -> 5.71 mm
- net N$7: track 5.08 -> 5.71 mm
- net N$6: track 5.08 -> 5.71 mm
- net N$5: track 5.08 -> 5.71 mm
- net N$4: track 5.08 -> 5.71 mm
- net N$3: track 5.08 -> 5.71 mm
- net N$30: track 5.08 -> 5.71 mm
- net N$29: track 5.08 -> 5.71 mm
- net N$28: track 5.08 -> 5.71 mm
- net N$26: track 5.08 -> 5.71 mm
- net N$25: track 5.08 -> 5.71 mm
- net N$23: track 5.08 -> 5.71 mm
- net N$20: track 5.08 -> 5.71 mm
- net N$2: track 5.08 -> 5.71 mm
- net N$19: track 5.08 -> 5.71 mm
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