File: EAGLE/MainBoard/V0_2/AVRI2CIO_V0_2_LEVEL0.sch (EAGLE design)
At the start: 38 parts

Commit message: update eagle files
Parts:
- X10: device con-wago-500:W237-102 -> con-wago-508:W237-02P; MPN 237-102 -> (none); OC_NEWARK 70K9898 -> (none)
- X11, X12, X13, X14, X15, X3, X4, X5, X6, X7, X8: device con-wago-500:W237-102 -> con-wago-508:W237-02P
Changed lines of the file:
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@@
 <?xml version="1.0" encoding="utf-8"?>
 <!DOCTYPE eagle SYSTEM "eagle.dtd">
-<eagle version="6.5.0">
+<eagle version="6.6.0">
 <drawing>
 <settings>
@@
 <part name="PH3_I" library="pinhead" deviceset="PINHD-1X5" device=""/>
 <part name="PH4_I" library="pinhead" deviceset="PINHD-1X5" device=""/>
-<part name="X3" library="con-wago-500" deviceset="W237-102" device=""/>
-<part name="X4" library="con-wago-500" deviceset="W237-102" device=""/>
-<part name="X5" library="con-wago-500" deviceset="W237-102" device=""/>
-<part name="X6" library="con-wago-500" deviceset="W237-102" device=""/>
-<part name="X7" library="con-wago-500" deviceset="W237-102" device=""/>
-<part name="X8" library="con-wago-500" deviceset="W237-102" device=""/>
+<part name="X3" library="con-wago-508" deviceset="W237-02P" device=""/>
+<part name="X4" library="con-wago-508" deviceset="W237-02P" device=""/>
+<part name="X5" library="con-wago-508" deviceset="W237-02P" device=""/>
+<part name="X6" library="con-wago-508" deviceset="W237-02P" device=""/>
+<part name="X7" library="con-wago-508" deviceset="W237-02P" device=""/>
+<part name="X8" library="con-wago-508" deviceset="W237-02P" device=""/>
 <part name="PH6_E" library="pinhead" deviceset="PINHD-1X3" device=""/>
 <part name="PH7_E" library="pinhead" deviceset="PINHD-1X3" device=""/>
@@
 <part name="PH4_E" library="pinhead" deviceset="PINHD-1X3" device=""/>
 <part name="PH5_E" library="pinhead" deviceset="PINHD-1X3" device=""/>
-<part name="X11" library="con-wago-500" deviceset="W237-102" device=""/>
-<part name="X12" library="con-wago-500" deviceset="W237-102" device=""/>
-<part name="X13" library="con-wago-500" deviceset="W237-102" device=""/>
-<part name="X14" library="con-wago-500" deviceset="W237-102" device=""/>
-<part name="X15" library="con-wago-500" deviceset="W237-102" device=""/>
+<part name="X11" library="con-wago-508" deviceset="W237-02P" device=""/>
+<part name="X12" library="con-wago-508" deviceset="W237-02P" device=""/>
+<part name="X13" library="con-wago-508" deviceset="W237-02P" device=""/>
+<part name="X14" library="con-wago-508" deviceset="W237-02P" device=""/>
+<part name="X15" library="con-wago-508" deviceset="W237-02P" device=""/>
 <part name="GND2" library="supply1" deviceset="GND" device=""/>
 <part name="GND3" library="supply1" deviceset="GND" device=""/>
@@
 <part name="GND25" library="supply1" deviceset="GND" device=""/>
 <part name="PH0_E" library="pinhead" deviceset="PINHD-1X3" device=""/>
-<part name="X10" library="con-wago-500" deviceset="W237-102" device="">
+<part name="X10" library="con-wago-508" deviceset="W237-02P" device="">
 <attribute name="MF" value=""/>
-<attribute name="MPN" value="237-102"/>
 <attribute name="OC_FARNELL" value="unknown"/>
-<attribute name="OC_NEWARK" value="70K9898"/>
 </part>
 <part name="GND1" library="supply1" deviceset="GND" device=""/>
